File: core_board/Power_in.kicad_sch (KiCad schematic)
At the start: 25 parts, among them J1 Molex_Megafit_02, Q1 TPC8132_LQS, U1 AP63205QWU7, U2 AP63301WU7

Commit message: Add temp sensor datasheet
Parts:
- added C12: 100nF, MRDT_Shields:RoveNode_H5, symbol Device:C
- added R8: 10kohm, Package_SO:TSSOP-20_4.4x6.5mm_P0.65mm, symbol Device:R_US
- added TH: Thermistor_NTC, Package_DFN_QFN:Nordic_AQFN-94-1EP_7x7mm_P0.4mm, symbol Device:Thermistor_NTC
Connections:
- net GND: now also C12.2, TH.2
- new net +3V3: R8.1
- new net TEMP_OUT: C12.1, R8.2, TH.1
Other:
- note added: "TEMP SENSOR"
